File: double-tuned-bpf.sch (KiCad schematic (older format))
At the start: 12 parts, among them J1 PCB_SMA_EDGE, J2 PCB_SMA_EDGE, J3 Conn_01x03_Female, J4 Conn_01x03_Female, T1 6:31, T2 31:6

Commit message: gg
Parts:
- C2, C3, C4, C5: symbol Tayloe-Mixer-v2-rescue:Capacitor-Xenir -> double-tuned-bpf-rescue:Capacitor-Xenir-Tayloe-Mixer-v2-rescue
- J1, J2: symbol Xenir:PCB_SMA_EDGE -> double-tuned-bpf-rescue:PCB_SMA_EDGE-Xenir
- T1, T2: symbol Tayloe-Mixer-v2-rescue:T37_XFRM-Xenir -> double-tuned-bpf-rescue:T37_XFRM-Xenir-Tayloe-Mixer-v2-rescue
- VC1, VC6: symbol Tayloe-Mixer-v2-rescue:Trimcap-Xenir -> double-tuned-bpf-rescue:Trimcap-Xenir-Tayloe-Mixer-v2-rescue
Changed lines of the file:
@@
 	4400 2650 4500 2650
 $Comp
-L Tayloe-Mixer-v2-rescue:T37_XFRM-Xenir T2
+L double-tuned-bpf-rescue:T37_XFRM-Xenir-Tayloe-Mixer-v2-rescue T2
 U 1 1 5E9E9ADC
 P 5450 2500
@@
 $EndComp
 $Comp
-L Tayloe-Mixer-v2-rescue:Trimcap-Xenir VC6
+L double-tuned-bpf-rescue:Trimcap-Xenir-Tayloe-Mixer-v2-rescue VC6
 U 1 1 5E9E8F97
 P 4850 2550
@@
 $EndComp
 $Comp
-L Tayloe-Mixer-v2-rescue:Capacitor-Xenir C3
+L double-tuned-bpf-rescue:Capacitor-Xenir-Tayloe-Mixer-v2-rescue C3
 U 1 1 5E9E8D24
 P 4250 2150
@@
 $EndComp
 $Comp
-L Tayloe-Mixer-v2-rescue:Capacitor-Xenir C4
+L double-tuned-bpf-rescue:Capacitor-Xenir-Tayloe-Mixer-v2-rescue C4
 U 1 1 5E9E81AF
 P 4250 2650
@@
 $EndComp
 $Comp
-L Tayloe-Mixer-v2-rescue:Capacitor-Xenir C5
+L double-tuned-bpf-rescue:Capacitor-Xenir-Tayloe-Mixer-v2-rescue C5
 U 1 1 5E9E7736
 P 4500 2950
@@
 $EndComp
 $Comp
-L Tayloe-Mixer-v2-rescue:Capacitor-Xenir C2
+L double-tuned-bpf-rescue:Capacitor-Xenir-Tayloe-Mixer-v2-rescue C2
 U 1 1 5E9E667F
 P 4000 2950
@@
 $EndComp
 $Comp
-L Tayloe-Mixer-v2-rescue:Trimcap-Xenir VC1
+L double-tuned-bpf-rescue:Trimcap-Xenir-Tayloe-Mixer-v2-rescue VC1
 U 1 1 5E9DC9D6
 P 3650 2550
@@
 $EndComp
 $Comp
-L Tayloe-Mixer-v2-rescue:T37_XFRM-Xenir T1
+L double-tuned-bpf-rescue:T37_XFRM-Xenir-Tayloe-Mixer-v2-rescue T1
 U 1 1 5E9D7159
 P 3050 2500
@@
 $EndBitmap
 $Comp
-L Xenir:PCB_SMA_EDGE J1
+L double-tuned-bpf-rescue:PCB_SMA_EDGE-Xenir J1
 U 1 1 6393BB21
 P 2175 2450
@@
 $EndComp
 $Comp
-L Xenir:PCB_SMA_EDGE J2
+L double-tuned-bpf-rescue:PCB_SMA_EDGE-Xenir J2
 U 1 1 6393CE58
 P 6200 2450

Commit message: gg
Connections:
- net GND: now also J3.1 (Pin_1), J4.1 (Pin_1)
- net Input: now also J3.2 (Pin_2); no longer J3.1 (Pin_1)
- net Output: now also J4.2 (Pin_2); no longer J4.1 (Pin_1)
Changed lines of the file:
@@
 Text GLabel 5925 2650 1    50   Input ~ 0
 Output
-Text GLabel 2650 3825 0    50   Input ~ 0
+Text GLabel 2650 3925 0    50   Input ~ 0
 Input
 $Comp
@@
 	1    0    0    -1
 $EndComp
-Text GLabel 3750 3825 0    50   Input ~ 0
+Text GLabel 3750 3925 0    50   Input ~ 0
 Output
 $Comp
@@
 	1    0    0    -1
 $EndComp
+Wire Wire Line
+	3750 3825 3375 3825
+Wire Wire Line
+	3375 3825 3375 4025
+Wire Wire Line
+	3375 4025 3750 4025
+Connection ~ 3750 4025
+Wire Wire Line
+	2650 3825 2350 3825
+Wire Wire Line
+	2350 3825 2350 4025
+Wire Wire Line
+	2350 4025 2650 4025
+Connection ~ 2650 4025
 $EndSCHEMATC
